File: hardware/IRAM256A/f4.kicad_sch (KiCad schematic)
At the start: 37 parts

Commit message: Structure change + kicad 3d models updated
Parts:
- C1, C119, C16, C29, C61, C66, C67, C77, C80, C84, C85, C86, C87, C89: value (none) -> 100n; footprint (none) -> stmbl:C_0603
- C31, C32: value (none) -> 18p; footprint (none) -> stmbl:C_0603
- C64, C81: value (none) -> 1n; footprint (none) -> stmbl:C_0603
- C65, C88, C90: value (none) -> 2.2µ; footprint (none) -> stmbl:C_0603
- JP9: value (none) -> Jumper_NO_Small; footprint (none) -> stmbl:SOLDER_JUMPER
- L3: value (none) -> 220r 700mA; footprint (none) -> stmbl:R_0603
- P1: value (none) -> USB_OTG; footprint (none) -> stmbl:USB_Micro-B
- R1: value (none) -> 120; footprint (none) -> stmbl:R_0603
- R116: value (none) -> 10k; footprint (none) -> stmbl:R_0603
- R117, R121, R122, R153, R61: value (none) -> 1k; footprint (none) -> stmbl:R_0603
- U1, U20, U22, U23: value (none) -> USBLC6-4SC6; footprint (none) -> stmbl:SOT-23-6
- U26: value (none) -> STM32F405VG; footprint (none) -> TQFP100
- Y2: value (none) -> 8M; footprint (none) -> stmbl:Crystal_SMD_0503_4Pads
